Commit message: Add the Dexplore_Dexhand021 task and configs
- dexplore_dexhand021.py: left DexHand021 task; URDF mimic couplings applied
  to PD targets and reset states, Inspire-style collision filter
- dexhand021.yaml / train/rlg/dexhand021.yaml: 25 DOFs, mirrored objects,
  key/contact bodies in the human joint order
- make_dexhand021_urdf.py: drop the 1 mm pad collision boxes so fingertip
  contacts land on the distal links
- check_ur10_reachability.py: skip doorknob sequences, prefer the IK branch
  that keeps the arm highest, exit without the pinocchio/torch teardown crash

Smoke test: 256 envs, 107 motions, mean reward 4.3 -> 13.8 in 46 epochs.

Co-Authored-By: Claude Opus 5.5 <noreply@anthropic.com>

File: dexplore/data/assets/dexhand021/dexhand021_left.urdf (robot description, URDF)
Before this commit: robot dexhand021_left_sim, 33 links, 32 joints
Links:
- link l_f_link1_pad: geometry visual box size=0.012 0.001 0.006
- link l_f_link2_pad: geometry visual box size=0.012 0.001 0.006
- link l_f_link3_pad: geometry visual box size=0.012 0.001 0.006
- link l_f_link4_pad: geometry visual box size=0.012 0.001 0.006
- link l_f_link5_pad: geometry visual box size=0.012 0.001 0.006
